File: PCBs/PCB2.1.0/OptronV7_PCB.brd (EAGLE design)
At the start: 72.4 x 100 mm, 40 parts, among them J1 POWER_JACK

Commit message: PCB review updates
Parts:
- added RESET_R10K: (no value), SparkFun-Resistors:AXIAL-0.3
- moved CAP_1 14.2 mm to (27.9, 6.35)
- moved CAP_2 9.16 mm to (27.9, 3.81)
Connections:
- new net N$1: RESET_R10K.P$1, TCA.1.5
- net 5V: now also RESET_R10K.P$2
- net GND: now also TCA.1.6, TCA.1.7, TCA.1.8
- net MO5: now also 74A1.6; no longer 74A1.3
- net SCK5: now also 74A1.3; no longer 74A1.6
- net SCL5V: now also TCA.1.4; no longer TCA.1.3
- net SDA5V: now also TCA.1.3; no longer TCA.1.4
Routing:
- net SDA5V: track 26.5 -> 12.8 mm
- net SCL5V: track 22.2 -> 12.8 mm
- net 3V: track 163.5 -> 157.6 mm
- net GND: track 5.61 -> 0.00 mm
- net MO5: track 18.8 -> 24.2 mm
- net 5V: track 5.08 -> 0.00 mm
- net SCK5: track 23.2 -> 19.9 mm
- net N$1: track 0.00 -> 2.54 mm
- net SDA: track 94.0 -> 95.3 mm
- net SCL: track 87.1 -> 87.9 mm
